File: pcb/right_side.kicad_sch (KiCad schematic)
At the start: 148 parts, among them J2 USB_C_Receptacle_USB2.0_14P, SW49 SW_Push, SW50 SW_Push, SW51 SW_Push, SW52 SW_Push, SW53 SW_Push, SW54 SW_Push, SW55 SW_Push, SW56 SW_Push, SW57 SW_Push, SW58 SW_Push, SW59 SW_Push, SW60 SW_Push, SW61 SW_Push, SW62 SW_Push, SW63 SW_Push, SW64 SW_Push, SW65 SW_Push, SW66 SW_Push, SW67 SW_Push, SW68 SW_Push, SW69 SW_Push, SW70 SW_Push, SW71 SW_Push, SW72 SW_Push, SW73 SW_Push, SW74 SW_Push, SW75 SW_Push, SW76 SW_Push, SW77 SW_Push, SW78 SW_Push, SW79 SW_Push, SW80 SW_Push, SW81 SW_Push, SW82 SW_Push, SW83 SW_Push, SW84 SW_Push, SW85 SW_Push, SW86 SW_Push, SW87 SW_Push, SW88 SW_Push, SW89 SW_Push, SW90 SW_Push, SW91 SW_Push, SW92 SW_Push, SW93 SW_Push, SW94 SW_Push, SW95 SW_Push, SW96 SW_Push

Commit message: update
Parts:
- removed LED49, LED50, LED51, LED52, LED53, LED54, LED55, LED56, LED57, LED58, LED59, LED60, LED61, LED62, LED63, LED64, LED65, LED66, LED67, LED68, LED69, LED70, LED71, LED72, LED73, LED74, LED75, LED76, LED77, LED78, LED79, LED80, LED81, LED82, LED83, LED84, LED85, LED86, LED87, LED88, LED89, LED90, LED91, LED92, LED93, LED94, LED95, LED96: SK6812MINI, LED_SMD:LED_SK6812MINI_PLCC4_3.5x3.5mm_P1.75mm, symbol LED:SK6812MINI
- removed RZ2: RP2040-Zero, RP2040-Zero-Kicad:RP2040-Zero, symbol rp2040-zero:RP2040-Zero
- added LED49, LED50, LED51, LED52, LED53, LED54, LED55, LED56, LED57, LED58, LED59, LED60, LED61, LED62, LED63, LED64, LED65, LED66, LED67, LED68, LED69, LED70, LED71, LED72, LED73, LED74, LED75, LED76, LED77, LED78, LED79, LED80, LED81, LED82, LED83, LED84, LED85, LED86, LED87, LED88, LED89, LED90, LED91, LED92, LED93, LED94, LED95, LED96: SK6812MINI-E, SK6812MINI-E:SK6812_mini_e_flipable, symbol SK6812MINI-E:SK6812MINI-E
- added MCU2: rp2040-zero, RP2040-Zero:Untitled, symbol zzkeeb:MCU_rp2040-zero
- SW65, SW89, SW90, SW94: footprint MX_Hotswap:MX-Hotswap-1U -> MX_Hotswap:MX-Hotswap-1.25U
- SW73, SW95: footprint MX_Hotswap:MX-Hotswap-1U -> MX_Hotswap:MX-Hotswap-1.5U
- SW81, SW96: footprint MX_Hotswap:MX-Hotswap-1U -> MX_Hotswap:MX-Hotswap-1.75U
Connections:
- net +3.3V: now also LED49.1 (VDD), LED50.1 (VDD), LED51.1 (VDD), LED52.1 (VDD), LED53.1 (VDD), LED54.1 (VDD), LED55.1 (VDD), LED56.1 (VDD), LED57.1 (VDD), LED58.1 (VDD), LED59.1 (VDD), LED60.1 (VDD), LED61.1 (VDD), LED62.1 (VDD), LED63.1 (VDD), LED64.1 (VDD), LED65.1 (VDD), LED66.1 (VDD), LED67.1 (VDD), LED68.1 (VDD), LED69.1 (VDD), LED70.1 (VDD), LED71.1 (VDD), LED72.1 (VDD), LED73.1 (VDD), LED74.1 (VDD), LED75.1 (VDD), LED76.1 (VDD), LED77.1 (VDD), LED78.1 (VDD), LED79.1 (VDD), LED80.1 (VDD), LED81.1 (VDD), LED82.1 (VDD), LED83.1 (VDD), LED84.1 (VDD), LED85.1 (VDD), LED86.1 (VDD), LED87.1 (VDD), LED88.1 (VDD), LED89.1 (VDD), LED90.1 (VDD), LED91.1 (VDD), LED92.1 (VDD), LED93.1 (VDD), LED94.1 (VDD), LED95.1 (VDD), LED96.1 (VDD), MCU2.21 (3V3)
- net +5V: now also MCU2.23 (5V)
- net GND: now also LED49.3 (VSS), LED50.3 (VSS), LED51.3 (VSS), LED52.3 (VSS), LED53.3 (VSS), LED54.3 (VSS), LED55.3 (VSS), LED56.3 (VSS), LED57.3 (VSS), LED58.3 (VSS), LED59.3 (VSS), LED60.3 (VSS), LED61.3 (VSS), LED62.3 (VSS), LED63.3 (VSS), LED64.3 (VSS), LED65.3 (VSS), LED66.3 (VSS), LED67.3 (VSS), LED68.3 (VSS), LED69.3 (VSS), LED70.3 (VSS), LED71.3 (VSS), LED72.3 (VSS), LED73.3 (VSS), LED74.3 (VSS), LED75.3 (VSS), LED76.3 (VSS), LED77.3 (VSS), LED78.3 (VSS), LED79.3 (VSS), LED80.3 (VSS), LED81.3 (VSS), LED82.3 (VSS), LED83.3 (VSS), LED84.3 (VSS), LED85.3 (VSS), LED86.3 (VSS), LED87.3 (VSS), LED88.3 (VSS), LED89.3 (VSS), LED90.3 (VSS), LED91.3 (VSS), LED92.3 (VSS), LED93.3 (VSS), LED94.3 (VSS), LED95.3 (VSS), LED96.3 (VSS), MCU2.22 (GND)
- net R_COL1: now also MCU2.3 (2)
- net R_COL2: now also MCU2.4 (3)
- net R_COL3: now also MCU2.5 (4)
- net R_COL4: now also MCU2.6 (5)
- net R_COL5: now also MCU2.7 (6)
- net R_COL6: now also MCU2.8 (7)
- net R_COL7: now also MCU2.9 (8)
- net R_COL8: now also MCU2.10 (9)
- net R_ROW1: now also MCU2.11 (10)
- net R_ROW2: now also MCU2.12 (11)
- net R_ROW3: now also MCU2.13 (12)
- net R_ROW4: now also MCU2.14 (13)
- net R_ROW5: now also MCU2.15 (14)
- net R_ROW6: now also MCU2.16 (15)
- net R_RX: now also MCU2.2 (1)
- net R_TX: now also MCU2.1 (0)
- new net: LED83.2 (DOUT), LED84.4 (DIN)
- new net: LED82.2 (DOUT), LED83.4 (DIN)
- new net: LED52.2 (DOUT), LED53.4 (DIN)
- new net: LED51.2 (DOUT), LED52.4 (DIN)
- new net: LED71.2 (DOUT), LED72.4 (DIN)
- new net: LED68.2 (DOUT), LED69.4 (DIN)
- new net: LED67.2 (DOUT), LED68.4 (DIN)
- new net: LED86.2 (DOUT), LED87.4 (DIN)
- new net: LED85.2 (DOUT), LED86.4 (DIN)
- new net: LED80.2 (DOUT), LED81.4 (DIN)
- new net: LED79.2 (DOUT), LED80.4 (DIN)
- new net: LED81.2 (DOUT), LED82.4 (DIN)
- new net: LED93.2 (DOUT), LED94.4 (DIN)
- new net: LED92.2 (DOUT), LED93.4 (DIN)
- new net: LED56.2 (DOUT), LED57.4 (DIN)
- new net: LED55.2 (DOUT), LED56.4 (DIN)
- new net: LED59.2 (DOUT), LED60.4 (DIN)
- new net: LED58.2 (DOUT), LED59.4 (DIN)
- new net: LED69.2 (DOUT), LED70.4 (DIN)
- new net: LED74.2 (DOUT), LED75.4 (DIN)
- new net: LED73.2 (DOUT), LED74.4 (DIN)
- new net: LED62.2 (DOUT), LED63.4 (DIN)
- new net: LED61.2 (DOUT), LED62.4 (DIN)
- new net: LED50.2 (DOUT), LED51.4 (DIN)
- new net: LED49.2 (DOUT), LED50.4 (DIN)
- new net: LED94.2 (DOUT), LED95.4 (DIN)
- new net: LED89.2 (DOUT), LED90.4 (DIN)
- new net: LED88.2 (DOUT), LED89.4 (DIN)
- new net: LED77.2 (DOUT), LED78.4 (DIN)
- new net: LED76.2 (DOUT), LED77.4 (DIN)
- new net: LED54.2 (DOUT), LED55.4 (DIN)
- new net: LED53.2 (DOUT), LED54.4 (DIN)
- new net: LED63.2 (DOUT), LED64.4 (DIN)
- new net: LED84.2 (DOUT), LED85.4 (DIN)
- new net: LED66.2 (DOUT), LED67.4 (DIN)
- new net: LED65.2 (DOUT), LED66.4 (DIN)
- new net: LED60.2 (DOUT), LED61.4 (DIN)
- new net: LED95.2 (DOUT), LED96.4 (DIN)
- new net: LED91.2 (DOUT), LED92.4 (DIN)
- new net: LED64.2 (DOUT), LED65.4 (DIN)
- new net: LED90.2 (DOUT), LED91.4 (DIN)
- new net: LED75.2 (DOUT), LED76.4 (DIN)
- new net: LED78.2 (DOUT), LED79.4 (DIN)
- new net: LED70.2 (DOUT), LED71.4 (DIN)
- new net: LED87.2 (DOUT), LED88.4 (DIN)
- new net: LED57.2 (DOUT), LED58.4 (DIN)
- new net R_LED1: LED49.4 (DIN), MCU2.20 (29)
- new net R_LED2: LED73.4 (DIN), MCU2.19 (28)
- no-connect marks 6 -> 4
