File: pcb/SplitKeeb.kicad_pcb (KiCad board)
At the start: 2 copper layers, 290 parts, among them SW1 SW_Push, SW10 SW_Push, SW11 SW_Push, SW12 SW_Push, SW13 SW_Push, SW14 SW_Push, SW15 SW_Push, SW16 SW_Push, SW17 SW_Push, SW18 SW_Push, SW19 SW_Push, SW2 SW_Push, SW20 SW_Push, SW21 SW_Push, SW22 SW_Push, SW23 SW_Push, SW24 SW_Push, SW25 SW_Push, SW26 SW_Push, SW27 SW_Push, SW28 SW_Push, SW29 SW_Push, SW3 SW_Push, SW30 SW_Push, SW31 SW_Push, SW32 SW_Push, SW33 SW_Push, SW34 SW_Push, SW35 SW_Push, SW36 SW_Push, SW37 SW_Push, SW38 SW_Push, SW39 SW_Push, SW4 SW_Push, SW40 SW_Push, SW41 SW_Push, SW42 SW_Push, SW43 SW_Push, SW44 SW_Push, SW45 SW_Push, SW46 SW_Push, SW47 SW_Push, SW48 SW_Push, SW49 SW_Push, SW5 SW_Push, SW50 SW_Push, SW51 SW_Push, SW52 SW_Push, SW53 SW_Push, SW54 SW_Push, SW55 SW_Push, SW56 SW_Push, SW57 SW_Push, SW58 SW_Push, SW59 SW_Push, SW6 SW_Push, SW60 SW_Push, SW61 SW_Push, SW62 SW_Push, SW63 SW_Push, SW64 SW_Push, SW65 SW_Push, SW66 SW_Push, SW67 SW_Push, SW68 SW_Push, SW69 SW_Push, SW7 SW_Push, SW70 SW_Push, SW71 SW_Push, SW72 SW_Push, SW73 SW_Push, SW74 SW_Push, SW75 SW_Push, SW76 SW_Push, SW77 SW_Push, SW78 SW_Push, SW79 SW_Push, SW8 SW_Push, SW80 SW_Push, SW81 SW_Push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

Commit message: update
Parts:
- removed D49, D50, D51, D52, D53, D54, D55, D56, D57, D58, D59, D60, D61, D62, D63, D64, D65, D66, D67, D68, D69, D70, D71, D72, D73, D74, D75, D76, D77, D78, D79, D80, D81, D82, D83, D84, D85, D86, D87, D88, D89, D90, D91, D92, D93, D94, D95, D96: D, Diode_SMD:D_SOD-123
- removed LED49, LED50, LED51, LED52, LED53, LED54, LED55, LED56, LED57, LED58, LED59, LED60, LED61, LED62, LED63, LED64, LED65, LED66, LED67, LED68, LED69, LED70, LED71, LED72, LED73, LED74, LED75, LED76, LED77, LED78, LED79, LED80, LED81, LED82, LED83, LED84, LED85, LED86, LED87, LED88, LED89, LED90, LED91, LED92, LED93, LED94, LED95, LED96: SK6812MINI, LED_SMD:LED_SK6812MINI_PLCC4_3.5x3.5mm_P1.75mm
- removed RZ1, RZ2: RP2040-Zero, RP2040-Zero-Kicad:RP2040-Zero
- removed SW49, SW50, SW51, SW52, SW53, SW54, SW55, SW56, SW57, SW58, SW59, SW60, SW61, SW62, SW63, SW64, SW65, SW66, SW67, SW68, SW69, SW70, SW71, SW72, SW73, SW74, SW75, SW76, SW77, SW78, SW79, SW80, SW81, SW82, SW83, SW84, SW85, SW86, SW87, SW88, SW89, SW90, SW91, SW92, SW93, SW94, SW95, SW96: SW_Push, MX_Hotswap:MX-Hotswap-1U
- added C1: 0.1uF, Capacitor_SMD:C_1206_3216Metric_Pad1.33x1.80mm_HandSolder, F.Cu at (95.9, -62.0)
- added C10: 0.1uF, Capacitor_SMD:C_1206_3216Metric_Pad1.33x1.80mm_HandSolder, F.Cu at (95.9, -31.8)
- added C11: 0.1uF, Capacitor_SMD:C_1206_3216Metric_Pad1.33x1.80mm_HandSolder, F.Cu at (95.9, -28.5)
- added C12: 0.1uF, Capacitor_SMD:C_1206_3216Metric_Pad1.33x1.80mm_HandSolder, F.Cu at (101.9, -62.0)
- added C13: 0.1uF, Capacitor_SMD:C_1206_3216Metric_Pad1.33x1.80mm_HandSolder, F.Cu at (101.9, -58.6)
- added C14: 0.1uF, Capacitor_SMD:C_1206_3216Metric_Pad1.33x1.80mm_HandSolder, F.Cu at (101.9, -55.3)
- added C15: 0.1uF, Capacitor_SMD:C_1206_3216Metric_Pad1.33x1.80mm_HandSolder, F.Cu at (101.9, -51.9)
- added C16: 0.1uF, Capacitor_SMD:C_1206_3216Metric_Pad1.33x1.80mm_HandSolder, F.Cu at (101.9, -48.6)
- added C17: 0.1uF, Capacitor_SMD:C_1206_3216Metric_Pad1.33x1.80mm_HandSolder, F.Cu at (101.9, -45.2)
- added C18: 0.1uF, Capacitor_SMD:C_1206_3216Metric_Pad1.33x1.80mm_HandSolder, F.Cu at (101.9, -41.9)
- added C19: 0.1uF, Capacitor_SMD:C_1206_3216Metric_Pad1.33x1.80mm_HandSolder, F.Cu at (101.9, -38.5)
- added C2: 0.1uF, Capacitor_SMD:C_1206_3216Metric_Pad1.33x1.80mm_HandSolder, F.Cu at (95.9, -58.6)
- added C20: 0.1uF, Capacitor_SMD:C_1206_3216Metric_Pad1.33x1.80mm_HandSolder, F.Cu at (101.9, -35.2)
- added C21: 0.1uF, Capacitor_SMD:C_1206_3216Metric_Pad1.33x1.80mm_HandSolder, F.Cu at (101.9, -31.8)
- added C22: 0.1uF, Capacitor_SMD:C_1206_3216Metric_Pad1.33x1.80mm_HandSolder, F.Cu at (101.9, -28.5)
- added C23: 0.1uF, Capacitor_SMD:C_1206_3216Metric_Pad1.33x1.80mm_HandSolder, F.Cu at (108.0, -62.0)
- added C24: 0.1uF, Capacitor_SMD:C_1206_3216Metric_Pad1.33x1.80mm_HandSolder, F.Cu at (108.0, -58.6)
- added C25: 0.1uF, Capacitor_SMD:C_1206_3216Metric_Pad1.33x1.80mm_HandSolder, F.Cu at (108.0, -55.3)
- added C26: 0.1uF, Capacitor_SMD:C_1206_3216Metric_Pad1.33x1.80mm_HandSolder, F.Cu at (108.0, -51.9)
- added C27: 0.1uF, Capacitor_SMD:C_1206_3216Metric_Pad1.33x1.80mm_HandSolder, F.Cu at (108.0, -48.6)
- added C28: 0.1uF, Capacitor_SMD:C_1206_3216Metric_Pad1.33x1.80mm_HandSolder, F.Cu at (108.0, -45.2)
- added C29: 0.1uF, Capacitor_SMD:C_1206_3216Metric_Pad1.33x1.80mm_HandSolder, F.Cu at (108.0, -41.9)
- added C3: 0.1uF, Capacitor_SMD:C_1206_3216Metric_Pad1.33x1.80mm_HandSolder, F.Cu at (95.9, -55.3)
- added C30: 0.1uF, Capacitor_SMD:C_1206_3216Metric_Pad1.33x1.80mm_HandSolder, F.Cu at (108.0, -38.5)
- added C31: 0.1uF, Capacitor_SMD:C_1206_3216Metric_Pad1.33x1.80mm_HandSolder, F.Cu at (108.0, -35.2)
- added C32: 0.1uF, Capacitor_SMD:C_1206_3216Metric_Pad1.33x1.80mm_HandSolder, F.Cu at (108.0, -31.8)
- added C33: 0.1uF, Capacitor_SMD:C_1206_3216Metric_Pad1.33x1.80mm_HandSolder, F.Cu at (108.0, -28.5)
- added C34: 0.1uF, Capacitor_SMD:C_1206_3216Metric_Pad1.33x1.80mm_HandSolder, F.Cu at (114.0, -62.0)
- added C35: 0.1uF, Capacitor_SMD:C_1206_3216Metric_Pad1.33x1.80mm_HandSolder, F.Cu at (114.0, -58.6)
- added C36: 0.1uF, Capacitor_SMD:C_1206_3216Metric_Pad1.33x1.80mm_HandSolder, F.Cu at (114.0, -55.3)
- added C37: 0.1uF, Capacitor_SMD:C_1206_3216Metric_Pad1.33x1.80mm_HandSolder, F.Cu at (114.0, -51.9)
- added C38: 0.1uF, Capacitor_SMD:C_1206_3216Metric_Pad1.33x1.80mm_HandSolder, F.Cu at (114.0, -48.6)
- added C39: 0.1uF, Capacitor_SMD:C_1206_3216Metric_Pad1.33x1.80mm_HandSolder, F.Cu at (114.0, -45.2)
- added C4: 0.1uF, Capacitor_SMD:C_1206_3216Metric_Pad1.33x1.80mm_HandSolder, F.Cu at (95.9, -51.9)
- added C40: 0.1uF, Capacitor_SMD:C_1206_3216Metric_Pad1.33x1.80mm_HandSolder, F.Cu at (114.0, -41.9)
- added C41: 0.1uF, Capacitor_SMD:C_1206_3216Metric_Pad1.33x1.80mm_HandSolder, F.Cu at (114.0, -38.5)
- added C42: 0.1uF, Capacitor_SMD:C_1206_3216Metric_Pad1.33x1.80mm_HandSolder, F.Cu at (114.0, -35.2)
- added C43: 0.1uF, Capacitor_SMD:C_1206_3216Metric_Pad1.33x1.80mm_HandSolder, F.Cu at (114.0, -31.8)
- added C44: 0.1uF, Capacitor_SMD:C_1206_3216Metric_Pad1.33x1.80mm_HandSolder, F.Cu at (114.0, -28.5)
- added C45: 0.1uF, Capacitor_SMD:C_1206_3216Metric_Pad1.33x1.80mm_HandSolder, F.Cu at (120.0, -62.0)
- added C46: 0.1uF, Capacitor_SMD:C_1206_3216Metric_Pad1.33x1.80mm_HandSolder, F.Cu at (120.0, -58.6)
- added C47: 0.1uF, Capacitor_SMD:C_1206_3216Metric_Pad1.33x1.80mm_HandSolder, F.Cu at (120.0, -55.3)
- added C48: 0.1uF, Capacitor_SMD:C_1206_3216Metric_Pad1.33x1.80mm_HandSolder, F.Cu at (120.0, -51.9)
- added C5: 0.1uF, Capacitor_SMD:C_1206_3216Metric_Pad1.33x1.80mm_HandSolder, F.Cu at (95.9, -48.6)
- added C6: 0.1uF, Capacitor_SMD:C_1206_3216Metric_Pad1.33x1.80mm_HandSolder, F.Cu at (95.9, -45.2)
- added C7: 0.1uF, Capacitor_SMD:C_1206_3216Metric_Pad1.33x1.80mm_HandSolder, F.Cu at (95.9, -41.9)
- added C8: 0.1uF, Capacitor_SMD:C_1206_3216Metric_Pad1.33x1.80mm_HandSolder, F.Cu at (95.9, -38.5)
- added C9: 0.1uF, Capacitor_SMD:C_1206_3216Metric_Pad1.33x1.80mm_HandSolder, F.Cu at (95.9, -35.2)
- added J1: USB_C_Receptacle_USB2.0_16P, PCM_marbastlib-various:USB_C_Receptacle_HRO_TYPE-C-31-M-12, F.Cu at (98.8, -21.0)
- added ShifterC1: C, Capacitor_SMD:C_1206_3216Metric_Pad1.33x1.80mm_HandSolder, F.Cu at (120.0, -48.6)
- added ShifterC2: C, Capacitor_SMD:C_1206_3216Metric_Pad1.33x1.80mm_HandSolder, F.Cu at (120.0, -45.2)
- added U1: MCU_rp2040-zero, RP2040-Zero:RP2040-Zero, F.Cu at (54.8, 49.9)
- added U2: SN74LV1T125DBV, Package_TO_SOT_SMD:SOT-23-5, F.Cu at (107.2, -24.4)
- added U3: SN74LV1T125DBV, Package_TO_SOT_SMD:SOT-23-5, F.Cu at (107.2, -19.8)
- LED1, LED10, LED11, LED12, LED13, LED14, LED15, LED16, LED17, LED18, LED19, LED2, LED20, LED21, LED22, LED23, LED24, LED25, LED26, LED27, LED28, LED29, LED3, LED30, LED31, LED32, LED33, LED34, LED35, LED36, LED37, LED38, LED39, LED4, LED40, LED41, LED42, LED43, LED44, LED45, LED46, LED47, LED48, LED5, LED6, LED7, LED8, LED9: value SK6812MINI -> MX_SK6812MINI-E; footprint LED_SMD:LED_SK6812MINI_PLCC4_3.5x3.5mm_P1.75mm -> PCM_marbastlib-mx:LED_MX_6028R
- SW1, SW10, SW11, SW12, SW13, SW14, SW15, SW16, SW18, SW19, SW2, SW20, SW21, SW22, SW23, SW24, SW26, SW27, SW28, SW29, SW3, SW30, SW31, SW32, SW34, SW35, SW36, SW37, SW38, SW39, SW4, SW40, SW43, SW44, SW45, SW5, SW6, SW7, SW8, SW9: footprint MX_Hotswap:MX-Hotswap-1U -> PCM_marbastlib-mx:SW_MX_HS_CPG151101S11_1u
- SW17, SW41, SW42, SW46: footprint MX_Hotswap:MX-Hotswap-1U -> PCM_marbastlib-mx:SW_MX_HS_CPG151101S11_1.25u
- SW25, SW47: footprint MX_Hotswap:MX-Hotswap-1U -> PCM_marbastlib-mx:SW_MX_HS_CPG151101S11_1.5u
- SW33, SW48: footprint MX_Hotswap:MX-Hotswap-1U -> PCM_marbastlib-mx:SW_MX_HS_CPG151101S11_1.75u
- moved LED45 937.1 mm to (88.6, -40.9)
- moved LED44 937.0 mm to (88.6, -46.0)
- moved LED43 937.0 mm to (88.6, -51.0)
- moved LED42 936.9 mm to (88.6, -56.1)
- moved LED41 936.9 mm to (88.6, -61.1)
- moved LED36 936.0 mm to (79.7, -35.9)
- moved LED35 936.0 mm to (79.7, -40.9)
- moved LED34 935.9 mm to (79.7, -46.0)
- moved LED33 935.9 mm to (79.7, -51.0)
- moved LED32 935.8 mm to (79.7, -56.1)
- moved LED31 935.8 mm to (79.7, -61.1)
- moved LED27 935.0 mm to (70.9, -30.8)
- moved LED26 934.9 mm to (70.9, -35.9)
- moved LED25 934.9 mm to (70.9, -40.9)
- moved LED24 934.8 mm to (70.9, -46.0)
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Connections:
- LED1 pad 1: Net-(LED1-DOUT) -> +5V
- LED1 pad 2: +3.3V -> Net-(LED1-DOUT)
- LED1 pad 3: L_LED -> L_LED1
- LED1 pad 4: +3.3V -> GND
- LED10 pad 1: Net-(LED10-DOUT) -> Net-(LED10-VDD)
- LED10 pad 2: +3.3V -> Net-(LED10-DOUT)
- LED10 pad 4: +3.3V -> GND
- LED11 pad 1: Net-(LED11-DOUT) -> Net-(LED10-VDD)
- LED11 pad 2: +3.3V -> Net-(LED10-DIN)
- LED11 pad 3: Net-(LED10-DOUT) -> Net-(LED11-DIN)
- LED11 pad 4: +3.3V -> GND
- LED12 pad 1: Net-(LED12-DOUT) -> Net-(LED10-VDD)
- LED12 pad 2: +3.3V -> Net-(LED11-DIN)
- LED12 pad 3: Net-(LED11-DOUT) -> Net-(LED12-DIN)
- LED12 pad 4: +3.3V -> GND
- LED13 pad 1: Net-(LED13-DOUT) -> Net-(LED10-VDD)
- LED13 pad 2: +3.3V -> Net-(LED12-DIN)
- LED13 pad 3: Net-(LED12-DOUT) -> Net-(LED13-DIN)
- LED13 pad 4: +3.3V -> GND
- LED14 pad 1: Net-(LED14-DOUT) -> Net-(LED10-VDD)
- LED14 pad 2: +3.3V -> Net-(LED13-DIN)
- LED14 pad 3: Net-(LED13-DOUT) -> Net-(LED14-DIN)
- LED14 pad 4: +3.3V -> GND
- LED15 pad 1: Net-(LED15-DOUT) -> Net-(LED10-VDD)
- LED15 pad 2: +3.3V -> Net-(LED14-DIN)
- LED15 pad 3: Net-(LED14-DOUT) -> Net-(LED15-DIN)
- LED15 pad 4: +3.3V -> GND
- LED16 pad 1: Net-(LED16-DOUT) -> Net-(LED10-VDD)
- LED16 pad 2: +3.3V -> Net-(LED15-DIN)
- LED16 pad 3: Net-(LED15-DOUT) -> Net-(LED16-DIN)
- LED16 pad 4: +3.3V -> GND
- LED17 pad 1: Net-(LED17-DOUT) -> +5V
- LED17 pad 2: +3.3V -> Net-(LED17-DOUT)
- LED17 pad 3: Net-(LED16-DOUT) -> Net-(LED17-DIN)
- LED17 pad 4: +3.3V -> GND
- LED18 pad 1: Net-(LED18-DOUT) -> +5V
- LED18 pad 2: +3.3V -> Net-(LED18-DOUT)
- LED18 pad 4: +3.3V -> GND
- LED19 pad 1: Net-(LED19-DOUT) -> +5V
- LED19 pad 2: +3.3V -> Net-(LED19-DOUT)
- LED19 pad 4: +3.3V -> GND
- LED2 pad 1: Net-(LED2-DOUT) -> +5V
- LED2 pad 2: +3.3V -> Net-(LED2-DOUT)
- LED2 pad 4: +3.3V -> GND
- LED20 pad 1: Net-(LED20-DOUT) -> +5V
- LED20 pad 2: +3.3V -> Net-(LED20-DOUT)
- LED20 pad 4: +3.3V -> GND
- LED21 pad 1: Net-(LED21-DOUT) -> +5V
- LED21 pad 2: +3.3V -> Net-(LED21-DOUT)
- LED21 pad 4: +3.3V -> GND
- LED22 pad 1: Net-(LED22-DOUT) -> +5V
- LED22 pad 2: +3.3V -> Net-(LED22-DOUT)
- LED22 pad 4: +3.3V -> GND
- LED23 pad 1: Net-(LED23-DOUT) -> +5V
- LED23 pad 2: +3.3V -> Net-(LED23-DOUT)
- LED23 pad 4: +3.3V -> GND
- LED24 pad 1: Net-(LED24-DOUT) -> +5V
- LED24 pad 2: +3.3V -> unconnected-(LED24-DOUT-Pad2)
- LED24 pad 4: +3.3V -> GND
- LED25 pad 1: Net-(LED25-DOUT) -> +5V
- LED25 pad 2: +3.3V -> Net-(LED25-DOUT)
- LED25 pad 3: Net-(LED24-DOUT) -> L_LED2
- LED25 pad 4: +3.3V -> GND
- LED26 pad 1: Net-(LED26-DOUT) -> +5V
- LED26 pad 2: +3.3V -> Net-(LED26-DOUT)
- LED26 pad 4: +3.3V -> GND
- LED27 pad 1: Net-(LED27-DOUT) -> +5V
- LED27 pad 2: +3.3V -> Net-(LED27-DOUT)
- LED27 pad 4: +3.3V -> GND
- LED28 pad 1: Net-(LED28-DOUT) -> +5V
- LED28 pad 2: +3.3V -> Net-(LED28-DOUT)
- LED28 pad 4: +3.3V -> GND
- LED29 pad 1: Net-(LED29-DOUT) -> +5V
- LED29 pad 2: +3.3V -> Net-(LED29-DOUT)
- LED29 pad 4: +3.3V -> GND
- LED3 pad 1: Net-(LED3-DOUT) -> +5V
- LED3 pad 2: +3.3V -> Net-(LED3-DOUT)
- LED3 pad 4: +3.3V -> GND
- LED30 pad 1: Net-(LED30-DOUT) -> +5V
- LED30 pad 2: +3.3V -> Net-(LED30-DOUT)
- LED30 pad 4: +3.3V -> GND
- LED31 pad 1: Net-(LED31-DOUT) -> +5V
- LED31 pad 2: +3.3V -> Net-(LED31-DOUT)
- LED31 pad 4: +3.3V -> GND
- LED32 pad 1: Net-(LED32-DOUT) -> +5V
- LED32 pad 2: +3.3V -> Net-(LED32-DOUT)
- LED32 pad 4: +3.3V -> GND
- LED33 pad 1: Net-(LED33-DOUT) -> Net-(LED33-VDD)
- LED33 pad 2: +3.3V -> Net-(LED33-DOUT)
- LED33 pad 3: Net-(LED32-DOUT) -> Net-(LED33-DIN)
- LED33 pad 4: +3.3V -> GND
- LED34 pad 1: Net-(LED34-DOUT) -> Net-(LED33-VDD)
- LED34 pad 2: +3.3V -> Net-(LED33-DIN)
- LED34 pad 3: Net-(LED33-DOUT) -> Net-(LED34-DIN)
- LED34 pad 4: +3.3V -> GND
- LED35 pad 1: Net-(LED35-DOUT) -> Net-(LED33-VDD)
- LED35 pad 2: +3.3V -> Net-(LED34-DIN)
- LED35 pad 3: Net-(LED34-DOUT) -> Net-(LED35-DIN)
- LED35 pad 4: +3.3V -> GND
- LED36 pad 1: Net-(LED36-DOUT) -> Net-(LED33-VDD)
- LED36 pad 2: +3.3V -> Net-(LED35-DIN)
- LED36 pad 3: Net-(LED35-DOUT) -> Net-(LED36-DIN)
- LED36 pad 4: +3.3V -> GND
- LED37 pad 1: Net-(LED37-DOUT) -> Net-(LED33-VDD)
- LED37 pad 2: +3.3V -> Net-(LED36-DIN)
- LED37 pad 3: Net-(LED36-DOUT) -> Net-(LED37-DIN)
- LED37 pad 4: +3.3V -> GND
- LED38 pad 1: Net-(LED38-DOUT) -> Net-(LED33-VDD)
- LED38 pad 2: +3.3V -> Net-(LED37-DIN)
- LED38 pad 3: Net-(LED37-DOUT) -> Net-(LED38-DIN)
- LED38 pad 4: +3.3V -> GND
- LED39 pad 1: Net-(LED39-DOUT) -> Net-(LED33-VDD)
- LED39 pad 2: +3.3V -> Net-(LED38-DIN)
- LED39 pad 3: Net-(LED38-DOUT) -> Net-(LED39-DIN)
- LED39 pad 4: +3.3V -> GND
- LED4 pad 1: Net-(LED4-DOUT) -> +5V
- LED4 pad 2: +3.3V -> Net-(LED4-DOUT)
- LED4 pad 4: +3.3V -> GND
- LED40 pad 1: Net-(LED40-DOUT) -> Net-(LED33-VDD)
- LED40 pad 2: +3.3V -> Net-(LED39-DIN)
- LED40 pad 3: Net-(LED39-DOUT) -> Net-(LED32-DOUT)
- LED40 pad 4: +3.3V -> GND
- LED41 pad 1: Net-(LED41-DOUT) -> +5V
- LED41 pad 2: +3.3V -> Net-(LED41-DOUT)
- LED41 pad 3: Net-(LED40-DOUT) -> Net-(LED33-DOUT)
- LED41 pad 4: +3.3V -> GND
- LED42 pad 1: Net-(LED42-DOUT) -> +5V
- LED42 pad 2: +3.3V -> Net-(LED42-DOUT)
- LED42 pad 4: +3.3V -> GND
- LED43 pad 1: Net-(LED43-DOUT) -> +5V
- LED43 pad 2: +3.3V -> Net-(LED43-DOUT)
- LED43 pad 4: +3.3V -> GND
- LED44 pad 1: Net-(LED44-DOUT) -> +5V
- LED44 pad 2: +3.3V -> Net-(LED44-DOUT)
- LED44 pad 4: +3.3V -> GND
- LED45 pad 1: Net-(LED45-DOUT) -> +5V
- LED45 pad 2: +3.3V -> Net-(LED45-DOUT)
- LED45 pad 4: +3.3V -> GND
- LED46 pad 1: Net-(LED46-DOUT) -> +5V
- LED46 pad 2: +3.3V -> Net-(LED46-DOUT)
- LED46 pad 4: +3.3V -> GND
- LED47 pad 1: Net-(LED47-DOUT) -> +5V
- LED47 pad 2: +3.3V -> Net-(LED47-DOUT)
- LED47 pad 4: +3.3V -> GND
- LED48 pad 1: unconnected-(LED48-DOUT-Pad1) -> +5V
- LED48 pad 2: +3.3V -> unconnected-(LED48-DOUT-Pad2)
- LED48 pad 4: +3.3V -> GND
- LED5 pad 1: Net-(LED5-DOUT) -> +5V
- LED5 pad 2: +3.3V -> Net-(LED5-DOUT)
- LED5 pad 4: +3.3V -> GND
- LED6 pad 1: Net-(LED6-DOUT) -> +5V
- LED6 pad 2: +3.3V -> Net-(LED6-DOUT)
- LED6 pad 4: +3.3V -> GND
- LED7 pad 1: Net-(LED7-DOUT) -> +5V
- LED7 pad 2: +3.3V -> Net-(LED7-DOUT)
- LED7 pad 4: +3.3V -> GND
- LED8 pad 1: Net-(LED8-DOUT) -> +5V
- LED8 pad 2: +3.3V -> Net-(LED16-DIN)
- LED8 pad 4: +3.3V -> GND
- LED9 pad 1: Net-(LED10-DIN) -> Net-(LED10-VDD)
- LED9 pad 2: +3.3V -> Net-(LED17-DIN)
- LED9 pad 3: Net-(LED8-DOUT) -> Net-(LED10-DOUT)
- LED9 pad 4: +3.3V -> GND
Routing:
- net L_COL8: track 0.00 -> 313.6 mm
- net L_ROW6: track 0.00 -> 309.6 mm, vias 0 -> 3
- net L_COL7: track 0.00 -> 288.8 mm
- net L_COL6: track 0.00 -> 265.2 mm
- net L_ROW5: track 0.00 -> 249.4 mm, vias 0 -> 1
- net L_ROW4: track 0.00 -> 227.2 mm, vias 0 -> 1
- net L_COL5: track 0.00 -> 220.9 mm
- net L_ROW3: track 0.00 -> 206.0 mm, vias 0 -> 1
- net L_COL4: track 0.00 -> 205.2 mm
- net L_COL3: track 0.00 -> 191.5 mm
- net L_ROW2: track 0.00 -> 183.5 mm, vias 0 -> 1
- net L_COL2: track 0.00 -> 179.1 mm
- net L_ROW1: track 0.00 -> 164.2 mm, vias 0 -> 1
- net L_COL1: track 0.00 -> 164.1 mm
- net Net-(D48-A): track 0.00 -> 9.99 mm
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- added copper zone on B.Cu, net GND
- added copper zone on F.Cu, net GND
Other:
- board outline added: 222.3 x 173.4 mm

Commit message: update pcb
Parts:
- removed the U2 at (107.2, -24.4)
- added ESD_C1: 10uF, Capacitor_SMD:C_0603_1608Metric_Pad1.08x0.95mm_HandSolder, F.Cu at (224.8, 75.1)
- added JP1: SolderJumper, Jumper:SolderJumper-3_P1.3mm_Open_RoundedPad1.0x1.5mm_NumberLabels, F.Cu at (215.9, 68.1)
- added JP2: SolderJumper, Jumper:SolderJumper-3_P1.3mm_Open_RoundedPad1.0x1.5mm_NumberLabels, F.Cu at (215.9, 72.7)
- added R1: 470, Resistor_SMD:R_0805_2012Metric_Pad1.20x1.40mm_HandSolder, F.Cu at (90.7, 55.1)
- added R2: 470, Resistor_SMD:R_0805_2012Metric_Pad1.20x1.40mm_HandSolder, F.Cu at (84.3, 133.3)
- added U1: SN74LV1T125DBV, Package_TO_SOT_SMD:SOT-23-5, F.Cu at (76.9, 56.5)
- added U4: SRV05-4, PCM_marbastlib-various:SOT-23-6-routable, F.Cu at (220.5, 75.3)
- C1, C10, C11, C12, C13, C14, C15, C16, C17, C18, C19, C2, C20, C21, C22, C23, C24, C25, C26, C27, C28, C29, C3, C30, C31, C32, C33, C34, C35, C36, C37, C38, C39, C4, C40, C41, C42, C43, C44, C45, C46, C47, C48, C5, C6, C7, C8, C9, ShifterC1, ShifterC2: footprint Capacitor_SMD:C_1206_3216Metric_Pad1.33x1.80mm_HandSolder -> Capacitor_SMD:C_0603_1608Metric_Pad1.08x0.95mm_HandSolder
- LED1, LED10, LED11, LED12, LED13, LED14, LED15, LED16, LED17, LED18, LED19, LED2, LED20, LED21, LED22, LED23, LED24, LED25, LED26, LED27, LED28, LED29, LED3, LED30, LED31, LED32, LED33, LED34, LED35, LED36, LED37, LED38, LED39, LED4, LED40, LED41, LED42, LED43, LED44, LED45, LED46, LED47, LED48, LED5, LED6, LED7, LED8, LED9: footprint PCM_marbastlib-mx:LED_MX_6028R -> PCM_marbastlib-mx:LED_MX_6028R-ROT
- moved C48 274.1 mm to (232.9, 197.9), turned to 75 degrees
- moved C47 266.6 mm to (214.2, 194.1), turned to 75 degrees
- moved LED48 264.5 mm to (237.5, 192.9), turned to -15 degrees
- moved C46 259.4 mm to (195.2, 189.6), turned to 75 degrees
- moved LED47 255.6 mm to (219.0, 189.0), turned to -15 degrees
- moved LED46 247.5 mm to (200.4, 185.0), turned to -15 degrees
- moved LED41 235.0 mm to (57.2, 171.8)
- moved LED32 233.8 mm to (216.6, 133.5)
- moved LED42 228.0 mm to (80.9, 171.8)
- moved LED31 227.9 mm to (197.8, 133.8)
- moved C45 224.2 mm to (136.1, 161.7), turned to 90 degrees
- moved C41 223.4 mm to (52.6, 176.3), turned to 90 degrees
- moved C40 222.0 mm to (213.6, 156.5), turned to 90 degrees
- moved LED43 218.4 mm to (102.3, 167.0)
- moved C39 217.1 mm to (194.6, 156.4), turned to 90 degrees
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- renumbered U1 to U2
Connections:
- C10 pad 2: Net-(LED10-VDD) -> +5V
- C11 pad 2: Net-(LED10-VDD) -> +5V
- C12 pad 2: Net-(LED10-VDD) -> +5V
- C13 pad 2: Net-(LED10-VDD) -> +5V
- C14 pad 2: Net-(LED10-VDD) -> +5V
- C15 pad 2: Net-(LED10-VDD) -> +5V
- C16 pad 2: Net-(LED10-VDD) -> +5V
- C33 pad 2: Net-(LED33-VDD) -> +5V
- C34 pad 2: Net-(LED33-VDD) -> +5V
- C35 pad 2: Net-(LED33-VDD) -> +5V
- C36 pad 2: Net-(LED33-VDD) -> +5V
- C37 pad 2: Net-(LED33-VDD) -> +5V
- C38 pad 2: Net-(LED33-VDD) -> +5V
- C39 pad 2: Net-(LED33-VDD) -> +5V
- C40 pad 2: Net-(LED33-VDD) -> +5V
- C9 pad 2: Net-(LED10-VDD) -> +5V
- J1 pad A4: +5V -> VSS_IN_FUSED
- J1 pad A6: L_TX -> LINK+
- J1 pad A7: L_RX -> LINK-
- J1 pad A9: +5V -> VSS_IN_FUSED
- J1 pad B4: +5V -> VSS_IN_FUSED
- J1 pad B6: L_TX -> LINK+
- J1 pad B7: L_RX -> LINK-
- J1 pad B9: +5V -> VSS_IN_FUSED
- LED10 pad 1: Net-(LED10-VDD) -> +5V
- LED11 pad 1: Net-(LED10-VDD) -> +5V
- LED12 pad 1: Net-(LED10-VDD) -> +5V
- LED13 pad 1: Net-(LED10-VDD) -> +5V
- LED14 pad 1: Net-(LED10-VDD) -> +5V
- LED15 pad 1: Net-(LED10-VDD) -> +5V
- LED16 pad 1: Net-(LED10-VDD) -> +5V
- LED33 pad 1: Net-(LED33-VDD) -> +5V
- LED34 pad 1: Net-(LED33-VDD) -> +5V
- LED35 pad 1: Net-(LED33-VDD) -> +5V
- LED36 pad 1: Net-(LED33-VDD) -> +5V
- LED37 pad 1: Net-(LED33-VDD) -> +5V
- LED38 pad 1: Net-(LED33-VDD) -> +5V
- LED39 pad 1: Net-(LED33-VDD) -> +5V
- LED40 pad 1: Net-(LED33-VDD) -> +5V
- LED9 pad 1: Net-(LED10-VDD) -> +5V
- ShifterC1 pad 1: GND -> +5V
- ShifterC1 pad 2: +5V -> GND
- ShifterC2 pad 1: +5V -> GND
- ShifterC2 pad 2: GND -> +5V
- U2 pad 1: L_TX -> USART_TX
- U2 pad 2: L_RX -> USART_RX
- U2 pad 21: +3.3V -> unconnected-(U2-3V3-Pad21)
- U3 pad 2: L_LED_3v3_1 -> L_LED_3v3_2
Routing:
- net GND: track 0.00 -> 1650.0 mm, vias 0 -> 95
- net +5V: track 0.00 -> 1434.9 mm, vias 0 -> 12
- net USART_TX: track 0.00 -> 190.3 mm, vias 0 -> 4
- net USART_RX: track 0.00 -> 178.9 mm, vias 0 -> 2
- net L_LED_3v3_2: track 0.00 -> 114.0 mm, vias 0 -> 2
- net Net-(LED45-DOUT): track 0.00 -> 109.6 mm, vias 0 -> 2
- net L_LED_3v3_1: track 0.00 -> 58.9 mm, vias 0 -> 1
- net Net-(LED16-DIN): track 0.00 -> 48.9 mm, vias 0 -> 2
- net Net-(LED23-DOUT): track 0.00 -> 46.4 mm, vias 0 -> 2
- net Net-(LED25-DOUT): track 0.00 -> 45.8 mm
- net Net-(LED17-DOUT): track 0.00 -> 43.8 mm
- net Net-(LED41-DOUT): track 0.00 -> 43.2 mm, vias 0 -> 2
- net Net-(LED42-DOUT): track 0.00 -> 43.1 mm
- net Net-(LED27-DOUT): track 0.00 -> 42.8 mm
- net Net-(LED19-DOUT): track 0.00 -> 42.3 mm
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Other:
- board size 222.3 x 173.4 mm -> 448.4 x 173.4 mm

Commit message: update left pcb
Parts:
- added ?: , , F.Cu at (228.5, 40.5)
- added ?: , , F.Cu at (56.8, 109.9)
- added ?: , , F.Cu at (246.0, 209.0)
- added ?: , , F.Cu at (40.5, 40.4)
- added ?: , , F.Cu at (184.0, 191.2)
- added ?: , , F.Cu at (83.4, 72.3)
- added ?: , , F.Cu at (197.7, 72.7)
- added ?: , , F.Cu at (151.3, 164.2)
- added ?: , , F.Cu at (183.8, 158.9)
- added ?: , , F.Cu at (257.9, 171.2)
- added ?: , , F.Cu at (111.8, 174.9)
- added ?: , , F.Cu at (40.5, 179.8)
- ShifterC1, ShifterC2: value C -> 0.1uF
Routing:
- net GND: track 1650.0 -> 1645.1 mm
- net +5V: track 1434.9 -> 1433.0 mm
Other:
- board size 448.4 x 173.4 mm -> 222.3 x 173.4 mm
