File: pcb/SplitKeeb.kicad_sch (KiCad schematic)
At the start: 0 parts

Commit message: update
Parts:
- added C1, C10, C11, C12, C13, C14, C15, C16, C17, C18, C19, C2, C20, C21, C22, C23, C24, C25, C26, C27, C28, C29, C3, C30, C31, C32, C33, C34, C35, C36, C37, C38, C39, C4, C40, C41, C42, C43, C44, C45, C46, C47, C48, C5, C6, C7, C8, C9: 0.1uF, Capacitor_SMD:C_1206_3216Metric_Pad1.33x1.80mm_HandSolder, symbol Device:C
- added D1, D10, D11, D12, D13, D14, D15, D16, D17, D18, D19, D2, D20, D21, D22, D23, D24, D25, D26, D27, D28, D29, D3, D30, D31, D32, D33, D34, D35, D36, D37, D38, D39, D4, D40, D41, D42, D43, D44, D45, D46, D47, D48, D5, D6, D7, D8, D9: D, Diode_SMD:D_SOD-123, symbol Device:D
- added ESD_C1: C, symbol Device:C
- added J1: USB_C_Receptacle_USB2.0_16P, PCM_marbastlib-various:USB_C_Receptacle_HRO_TYPE-C-31-M-12, symbol Connector:USB_C_Receptacle_USB2.0_16P
- added JP1: LINK-, prettylib:SOLDER_JUMPER_3, symbol YAEMK:SolderJumper_3_Open
- added JP2: LINK+, prettylib:SOLDER_JUMPER_3, symbol YAEMK:SolderJumper_3_Open
- added LED1, LED10, LED11, LED12, LED13, LED14, LED15, LED16, LED17, LED18, LED19, LED2, LED20, LED21, LED22, LED23, LED24, LED25, LED26, LED27, LED28, LED29, LED3, LED30, LED31, LED32, LED33, LED34, LED35, LED36, LED37, LED38, LED39, LED4, LED40, LED41, LED42, LED43, LED44, LED45, LED46, LED47, LED48, LED5, LED6, LED7, LED8, LED9: MX_SK6812MINI-E, PCM_marbastlib-mx:LED_MX_6028R, symbol PCM_marbastlib-mx:MX_SK6812MINI-E
- added R1, R2: 470, Resistor_SMD:R_0805_2012Metric_Pad1.20x1.40mm_HandSolder, symbol Device:R
- added SW1, SW10, SW11, SW12, SW13, SW14, SW15, SW16, SW18, SW19, SW2, SW20, SW21, SW22, SW23, SW24, SW26, SW27, SW28, SW29, SW3, SW30, SW31, SW32, SW34, SW35, SW36, SW37, SW38, SW39, SW4, SW40, SW43, SW44, SW45, SW5, SW6, SW7, SW8, SW9: SW_Push, PCM_marbastlib-mx:SW_MX_HS_CPG151101S11_1u, symbol Switch:SW_Push_45deg
- added SW17, SW41, SW42, SW46: SW_Push, PCM_marbastlib-mx:SW_MX_HS_CPG151101S11_1.25u, symbol Switch:SW_Push_45deg
- added SW25, SW47: SW_Push, PCM_marbastlib-mx:SW_MX_HS_CPG151101S11_1.5u, symbol Switch:SW_Push_45deg
- added SW33, SW48: SW_Push, PCM_marbastlib-mx:SW_MX_HS_CPG151101S11_1.75u, symbol Switch:SW_Push_45deg
- added ShifterC1, ShifterC2: C, Capacitor_SMD:C_1206_3216Metric_Pad1.33x1.80mm_HandSolder, symbol Device:C
- added U1: MCU_rp2040-zero, RP2040-Zero:RP2040-Zero, symbol RP2040-Zero:MCU_rp2040-zero
- added U2, U3: SN74LV1T125DBV, Package_TO_SOT_SMD:SOT-23-5, symbol Logic_LevelTranslator:SN74LV1T125DBV
- added U4: SRV0504, prettylib:SOT-23-6, symbol YAEMK:SRV0504
Connections:
- new net: D23.2 (A), SW23.2
- new net: LED46.2 (DOUT), LED47.3 (DIN)
- new net: LED45.2 (DOUT), LED46.3 (DIN)
- new net: D47.2 (A), SW47.2
- new net: D42.2 (A), SW42.2
- new net: LED29.2 (DOUT), LED30.3 (DIN)
- new net: LED28.2 (DOUT), LED29.3 (DIN)
- new net: D27.2 (A), SW27.2
- new net: LED44.2 (DOUT), LED45.3 (DIN)
- new net: LED43.2 (DOUT), LED44.3 (DIN)
- new net: D10.2 (A), SW10.2
- new net: LED4.2 (DOUT), LED5.3 (DIN)
- new net: LED3.2 (DOUT), LED4.3 (DIN)
- new net: D26.2 (A), SW26.2
- new net: LED5.2 (DOUT), LED6.3 (DIN)
- new net: D45.2 (A), SW45.2
- new net: LED37.3 (DIN), LED38.2 (DOUT)
- new net: LED38.3 (DIN), LED39.2 (DOUT)
- new net: D19.2 (A), SW19.2
- new net: LED15.3 (DIN), LED16.2 (DOUT)
- new net: LED16.3 (DIN), LED8.2 (DOUT)
- new net: LED19.2 (DOUT), LED20.3 (DIN)
- new net: LED18.2 (DOUT), LED19.3 (DIN)
- new net: LED17.2 (DOUT), LED18.3 (DIN)
- new net: LED17.3 (DIN), LED9.2 (DOUT)
- new net: D14.2 (A), SW14.2
- new net: LED2.2 (DOUT), LED3.3 (DIN)
- new net: LED1.2 (DOUT), LED2.3 (DIN)
- new net: D33.2 (A), SW33.2
- new net: D29.2 (A), SW29.2
- new net: R1.2, U3.4 (Y)
- new net: D41.2 (A), SW41.2
- new net: D39.2 (A), SW39.2
- new net: D3.2 (A), SW3.2
- new net: D11.2 (A), SW11.2
- new net: D38.2 (A), SW38.2
- new net: D12.2 (A), SW12.2
- new net: D2.2 (A), SW2.2
- new net: LED6.2 (DOUT), LED7.3 (DIN)
- new net: LED13.3 (DIN), LED14.2 (DOUT)
- new net: LED14.3 (DIN), LED15.2 (DOUT)
- new net: D30.2 (A), SW30.2
- new net: LED36.3 (DIN), LED37.2 (DOUT)
- new net: D8.2 (A), SW8.2
- new net: D5.2 (A), SW5.2
- new net: D22.2 (A), SW22.2
- new net: D21.2 (A), SW21.2
- new net: LED11.3 (DIN), LED12.2 (DOUT)
- new net: LED12.3 (DIN), LED13.2 (DOUT)
- new net: LED42.2 (DOUT), LED43.3 (DIN)
- new net: LED41.2 (DOUT), LED42.3 (DIN)
- new net: LED39.3 (DIN), LED40.2 (DOUT)
- new net: D37.2 (A), SW37.2
- new net: LED34.3 (DIN), LED35.2 (DOUT)
- new net: LED35.3 (DIN), LED36.2 (DOUT)
- new net: D20.2 (A), SW20.2
- new net: LED20.2 (DOUT), LED21.3 (DIN)
- new net: LED10.2 (DOUT), LED9.3 (DIN)
- new net: LED10.3 (DIN), LED11.2 (DOUT)
- new net: LED26.2 (DOUT), LED27.3 (DIN)
- new net: LED25.2 (DOUT), LED26.3 (DIN)
- new net: LED21.2 (DOUT), LED22.3 (DIN)
- new net: D7.2 (A), SW7.2
- new net: LED7.2 (DOUT), LED8.3 (DIN)
- new net: D46.2 (A), SW46.2
- new net: D15.2 (A), SW15.2
- new net: D6.2 (A), SW6.2
- new net: R2.2, U2.4 (Y)
- new net: D35.2 (A), SW35.2
- new net: D9.2 (A), SW9.2
- new net: D25.2 (A), SW25.2
- new net: D17.2 (A), SW17.2
- new net: D16.2 (A), SW16.2
- new net: D31.2 (A), SW31.2
- new net: D28.2 (A), SW28.2
- new net: LED33.2 (DOUT), LED41.3 (DIN)
- new net: LED47.2 (DOUT), LED48.3 (DIN)
- new net: D44.2 (A), SW44.2
- new net: LED27.2 (DOUT), LED28.3 (DIN)
- new net: D18.2 (A), SW18.2
- new net: D43.2 (A), SW43.2
- new net: D4.2 (A), SW4.2
- new net: LED32.2 (DOUT), LED40.3 (DIN)
- new net: LED31.2 (DOUT), LED32.3 (DIN)
- new net: D13.2 (A), SW13.2
- new net: D32.2 (A), SW32.2
- new net: D48.2 (A), SW48.2
- new net: D1.2 (A), SW1.2
- new net: LED22.2 (DOUT), LED23.3 (DIN)
- new net: D24.2 (A), SW24.2
- new net: LED33.3 (DIN), LED34.2 (DOUT)
- new net: D36.2 (A), SW36.2
- new net: D40.2 (A), SW40.2
- new net: LED23.2 (DOUT), LED24.3 (DIN)
- new net: D34.2 (A), SW34.2
- new net: LED30.2 (DOUT), LED31.3 (DIN)
- new net +3.3V: U1.21 (3V3)
- new net +5V: C1.2, C10.2, C11.2, C12.2, C13.2, C14.2, C15.2, C16.2, C17.2, C18.2, C19.2, C2.2, C20.2, C21.2, C22.2, C23.2, C24.2, C25.2, C26.2, C27.2, C28.2, C29.2, C3.2, C30.2, C31.2, C32.2, C33.2, C34.2, C35.2, C36.2, C37.2, C38.2, C39.2, C4.2, C40.2, C41.2, C42.2, C43.2, C44.2, C45.2, C46.2, C47.2, C48.2, C5.2, C6.2, C7.2, C8.2, C9.2, ESD_C1.1, LED1.1 (VDD), LED10.1 (VDD), LED11.1 (VDD), LED12.1 (VDD), LED13.1 (VDD), LED14.1 (VDD), LED15.1 (VDD), LED16.1 (VDD), LED17.1 (VDD), LED18.1 (VDD), LED19.1 (VDD), LED2.1 (VDD), LED20.1 (VDD), LED21.1 (VDD), LED22.1 (VDD), LED23.1 (VDD), LED24.1 (VDD), LED25.1 (VDD), LED26.1 (VDD), LED27.1 (VDD), LED28.1 (VDD), LED29.1 (VDD), LED3.1 (VDD), LED30.1 (VDD), LED31.1 (VDD), LED32.1 (VDD), LED33.1 (VDD), LED34.1 (VDD), LED35.1 (VDD), LED36.1 (VDD), LED37.1 (VDD), LED38.1 (VDD), LED39.1 (VDD), LED4.1 (VDD), LED40.1 (VDD), LED41.1 (VDD), LED42.1 (VDD), LED43.1 (VDD), LED44.1 (VDD), LED45.1 (VDD), LED46.1 (VDD), LED47.1 (VDD), LED48.1 (VDD), LED5.1 (VDD), LED6.1 (VDD), LED7.1 (VDD), LED8.1 (VDD), LED9.1 (VDD), ShifterC1.2, ShifterC2.1, U1.23 (5V), U2.5 (VCC), U3.5 (VCC), U4.2 (GND)
- new net GND: C1.1, C10.1, C11.1, C12.1, C13.1, C14.1, C15.1, C16.1, C17.1, C18.1, C19.1, C2.1, C20.1, C21.1, C22.1, C23.1, C24.1, C25.1, C26.1, C27.1, C28.1, C29.1, C3.1, C30.1, C31.1, C32.1, C33.1, C34.1, C35.1, C36.1, C37.1, C38.1, C39.1, C4.1, C40.1, C41.1, C42.1, C43.1, C44.1, C45.1, C46.1, C47.1, C48.1, C5.1, C6.1, C7.1, C8.1, C9.1, J1.A1 (GND), J1.A12 (GND), J1.B1 (GND), J1.B12 (GND), J1.S1 (SHIELD), LED1.4 (VSS), LED10.4 (VSS), LED11.4 (VSS), LED12.4 (VSS), LED13.4 (VSS), LED14.4 (VSS), LED15.4 (VSS), LED16.4 (VSS), LED17.4 (VSS), LED18.4 (VSS), LED19.4 (VSS), LED2.4 (VSS), LED20.4 (VSS), LED21.4 (VSS), LED22.4 (VSS), LED23.4 (VSS), LED24.4 (VSS), LED25.4 (VSS), LED26.4 (VSS), LED27.4 (VSS), LED28.4 (VSS), LED29.4 (VSS), LED3.4 (VSS), LED30.4 (VSS), LED31.4 (VSS), LED32.4 (VSS), LED33.4 (VSS), LED34.4 (VSS), LED35.4 (VSS), LED36.4 (VSS), LED37.4 (VSS), LED38.4 (VSS), LED39.4 (VSS), LED4.4 (VSS), LED40.4 (VSS), LED41.4 (VSS), LED42.4 (VSS), LED43.4 (VSS), LED44.4 (VSS), LED45.4 (VSS), LED46.4 (VSS), LED47.4 (VSS), LED48.4 (VSS), LED5.4 (VSS), LED6.4 (VSS), LED7.4 (VSS), LED8.4 (VSS), LED9.4 (VSS), ShifterC1.1, ShifterC2.2, U1.22 (GND), U2.1 (~{OE}), U2.3 (GND), U3.1 (~{OE}), U3.3 (GND)
- new net LINK+: J1.A6 (D+), J1.B6 (D+), JP2.2 (C), U4.3 (I/O2)
- new net LINK-: J1.A7 (D-), J1.B7 (D-), JP1.2 (C), U4.1 (I/O1)
- new net L_COL1: SW1.1, SW17.1, SW25.1, SW33.1, SW41.1, SW9.1, U1.10 (9)
- new net L_COL2: SW10.1, SW18.1, SW2.1, SW26.1, SW34.1, SW42.1, U1.9 (8)
- new net L_COL3: SW11.1, SW19.1, SW27.1, SW3.1, SW35.1, SW43.1, U1.8 (7)
- new net L_COL4: SW12.1, SW20.1, SW28.1, SW36.1, SW4.1, SW44.1, U1.7 (6)
- new net L_COL5: SW13.1, SW21.1, SW29.1, SW37.1, SW45.1, SW5.1, U1.6 (5)
- new net L_COL6: SW14.1, SW22.1, SW30.1, SW38.1, SW46.1, SW6.1, U1.5 (4)
- new net L_COL7: SW15.1, SW23.1, SW31.1, SW39.1, SW47.1, SW7.1, U1.4 (3)
- new net L_COL8: SW16.1, SW24.1, SW32.1, SW40.1, SW48.1, SW8.1, U1.3 (2)
- new net L_LED1: LED1.3 (DIN), R1.1
- new net L_LED2: LED25.3 (DIN), R2.1
- new net L_LED_3v3_1: U1.20 (29), U3.2 (A)
- new net L_LED_3v3_2: U1.19 (28), U2.2 (A)
- new net L_ROW1: D1.1 (K), D2.1 (K), D3.1 (K), D4.1 (K), D5.1 (K), D6.1 (K), D7.1 (K), D8.1 (K), U1.11 (10)
- new net L_ROW2: D10.1 (K), D11.1 (K), D12.1 (K), D13.1 (K), D14.1 (K), D15.1 (K), D16.1 (K), D9.1 (K), U1.12 (11)
- new net L_ROW3: D17.1 (K), D18.1 (K), D19.1 (K), D20.1 (K), D21.1 (K), D22.1 (K), D23.1 (K), D24.1 (K), U1.13 (12)
- new net L_ROW4: D25.1 (K), D26.1 (K), D27.1 (K), D28.1 (K), D29.1 (K), D30.1 (K), D31.1 (K), D32.1 (K), U1.14 (13)
- new net L_ROW5: D33.1 (K), D34.1 (K), D35.1 (K), D36.1 (K), D37.1 (K), D38.1 (K), D39.1 (K), D40.1 (K), U1.15 (14)
- new net L_ROW6: D41.1 (K), D42.1 (K), D43.1 (K), D44.1 (K), D45.1 (K), D46.1 (K), D47.1 (K), D48.1 (K), U1.16 (15)
- new net USART_RX: JP1.1 (A), JP1.3 (B), JP2.1 (A), JP2.3 (B), U1.2 (1)
- new net USART_TX: U1.1 (0)
- new net VSS_IN_FUSED: ESD_C1.2, J1.A4 (VBUS), J1.A9 (VBUS), J1.B4 (VBUS), J1.B9 (VBUS), U4.5 (VBUS)
- no-connect marks 0 -> 10
Other:
- removed sheet left
- removed sheet right

Commit message: update pcb
Parts:
- removed JP1: LINK-, prettylib:SOLDER_JUMPER_3, symbol YAEMK:SolderJumper_3_Open
- removed JP2: LINK+, prettylib:SOLDER_JUMPER_3, symbol YAEMK:SolderJumper_3_Open
- removed U4: SRV0504, prettylib:SOT-23-6, symbol YAEMK:SRV0504
- added JP1, JP2: SolderJumper, Jumper:SolderJumper-3_P1.3mm_Open_RoundedPad1.0x1.5mm_NumberLabels, symbol Jumper:SolderJumper_3_Open
- added U4: SRV05-4, PCM_marbastlib-various:SOT-23-6-routable, symbol PCM_marbastlib-various:SRV05-4
- C1, C10, C11, C12, C13, C14, C15, C16, C17, C18, C19, C2, C20, C21, C22, C23, C24, C25, C26, C27, C28, C29, C3, C30, C31, C32, C33, C34, C35, C36, C37, C38, C39, C4, C40, C41, C42, C43, C44, C45, C46, C47, C48, C5, C6, C7, C8, C9: footprint Capacitor_SMD:C_1206_3216Metric_Pad1.33x1.80mm_HandSolder -> Capacitor_SMD:C_0603_1608Metric_Pad1.08x0.95mm_HandSolder
- ESD_C1: value C -> 10uF; footprint (none) -> Capacitor_SMD:C_0603_1608Metric_Pad1.08x0.95mm_HandSolder
- LED1, LED10, LED11, LED12, LED13, LED14, LED15, LED16, LED17, LED18, LED19, LED2, LED20, LED21, LED22, LED23, LED24, LED25, LED26, LED27, LED28, LED29, LED3, LED30, LED31, LED32, LED33, LED34, LED35, LED36, LED37, LED38, LED39, LED4, LED40, LED41, LED42, LED43, LED44, LED45, LED46, LED47, LED48, LED5, LED6, LED7, LED8, LED9: footprint PCM_marbastlib-mx:LED_MX_6028R -> PCM_marbastlib-mx:LED_MX_6028R-ROT
- ShifterC1: renamed from ShifterC2; footprint Capacitor_SMD:C_1206_3216Metric_Pad1.33x1.80mm_HandSolder -> Capacitor_SMD:C_0603_1608Metric_Pad1.08x0.95mm_HandSolder
- ShifterC2: renamed from ShifterC1; footprint Capacitor_SMD:C_1206_3216Metric_Pad1.33x1.80mm_HandSolder -> Capacitor_SMD:C_0603_1608Metric_Pad1.08x0.95mm_HandSolder
- renumbered U3 to U1, U1 to U2, U2 to U3
Connections:
- net +5V: no longer ESD_C1.1
- net GND: now also ESD_C1.1, U4.2 (VN)
- net LINK+: now also JP1.2 (C), U4.6 (IO4)
- net LINK-: now also JP2.2 (C), U4.1 (IO1)
- net USART_RX: now also JP1.1 (A), JP2.1 (A)
- net USART_TX: now also JP1.3 (B), JP2.3 (B)
- net VSS_IN_FUSED: now also U4.5 (VP)
- net +3.3V: no longer names the net of U2.21 (3V3)
- no-connect marks 10 -> 11
Other:
- moved on the sheet: C1, C10, C11, C12, C13, C14, C15, C16, C17, C18, C19, C2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

Commit message: update left pcb
Parts:
- added C100, C101, C102, C103, C104, C105, C106, C107, C108, C109, C110, C111, C112, C113, C114, C115, C116, C117, C118, C119, C120, C121, C122, C123, C124, C125, C126, C127, C128, C129, C130, C131, C132, C133, C134, C135, C136, C137, C138, C139, C140, C141, C142, C143, C144, C97, C98, C99, ShifterC5, ShifterC6: 0.1uF, Capacitor_SMD:C_0603_1608Metric_Pad1.08x0.95mm_HandSolder, symbol Device:C
- added D100, D101, D102, D103, D104, D105, D106, D107, D108, D109, D110, D111, D112, D113, D114, D115, D116, D117, D118, D119, D120, D121, D122, D123, D124, D125, D126, D127, D128, D129, D130, D131, D132, D133, D134, D135, D136, D137, D138, D139, D140, D141, D142, D143, D144, D97, D98, D99: D, Diode_SMD:D_SOD-123, symbol Device:D
- added ESD_C3: 10uF, Capacitor_SMD:C_0603_1608Metric_Pad1.08x0.95mm_HandSolder, symbol Device:C
- added J3: USB_C_Receptacle_USB2.0_16P, PCM_marbastlib-various:USB_C_Receptacle_HRO_TYPE-C-31-M-12, symbol Connector:USB_C_Receptacle_USB2.0_16P
- added JP5, JP6: SolderJumper, Jumper:SolderJumper-3_P1.3mm_Open_RoundedPad1.0x1.5mm_NumberLabels, symbol Jumper:SolderJumper_3_Open
- added LED100, LED101, LED102, LED103, LED104, LED105, LED106, LED107, LED108, LED109, LED110, LED111, LED112, LED113, LED114, LED115, LED116, LED117, LED118, LED119, LED120, LED121, LED122, LED123, LED124, LED125, LED126, LED127, LED128, LED129, LED130, LED131, LED132, LED133, LED134, LED135, LED136, LED137, LED138, LED139, LED140, LED141, LED142, LED143, LED144, LED97, LED98, LED99: MX_SK6812MINI-E, PCM_marbastlib-mx:LED_MX_6028R-ROT, symbol PCM_marbastlib-mx:MX_SK6812MINI-E
- added R5, R6: 470, Resistor_SMD:R_0805_2012Metric_Pad1.20x1.40mm_HandSolder, symbol Device:R
- added SW100, SW101, SW102, SW103, SW104, SW105, SW106, SW107, SW108, SW109, SW110, SW111, SW112, SW114, SW115, SW116, SW117, SW118, SW119, SW120, SW122, SW123, SW124, SW125, SW126, SW127, SW128, SW130, SW131, SW132, SW133, SW134, SW135, SW136, SW139, SW140, SW141, SW97, SW98, SW99: SW_Push, PCM_marbastlib-mx:SW_MX_HS_CPG151101S11_1u, symbol Switch:SW_Push_45deg
- added SW113, SW137, SW138, SW142: SW_Push, PCM_marbastlib-mx:SW_MX_HS_CPG151101S11_1.25u, symbol Switch:SW_Push_45deg
- added SW121, SW143: SW_Push, PCM_marbastlib-mx:SW_MX_HS_CPG151101S11_1.5u, symbol Switch:SW_Push_45deg
- added SW129, SW144: SW_Push, PCM_marbastlib-mx:SW_MX_HS_CPG151101S11_1.75u, symbol Switch:SW_Push_45deg
- added U10: MCU_rp2040-zero, RP2040-Zero:RP2040-Zero, symbol RP2040-Zero:MCU_rp2040-zero
- added U11, U9: SN74LV1T125DBV, Package_TO_SOT_SMD:SOT-23-5, symbol Logic_LevelTranslator:SN74LV1T125DBV
- added U12: SRV05-4, PCM_marbastlib-various:SOT-23-6-routable, symbol PCM_marbastlib-various:SRV05-4
- ShifterC1, ShifterC2: value C -> 0.1uF
Connections:
- net +5V: now also C100.2, C101.2, C102.2, C103.2, C104.2, C105.2, C106.2, C107.2, C108.2, C109.2, C110.2, C111.2, C112.2, C113.2, C114.2, C115.2, C116.2, C117.2, C118.2, C119.2, C120.2, C121.2, C122.2, C123.2, C124.2, C125.2, C126.2, C127.2, C128.2, C129.2, C130.2, C131.2, C132.2, C133.2, C134.2, C135.2, C136.2, C137.2, C138.2, C139.2, C140.2, C141.2, C142.2, C143.2, C144.2, C97.2, C98.2, C99.2, LED100.1 (VDD), LED101.1 (VDD), LED102.1 (VDD), LED103.1 (VDD), LED104.1 (VDD), LED105.1 (VDD), LED106.1 (VDD), LED107.1 (VDD), LED108.1 (VDD), LED109.1 (VDD), LED110.1 (VDD), LED111.1 (VDD), LED112.1 (VDD), LED113.1 (VDD), LED114.1 (VDD), LED115.1 (VDD), LED116.1 (VDD), LED117.1 (VDD), LED118.1 (VDD), LED119.1 (VDD), LED120.1 (VDD), LED121.1 (VDD), LED122.1 (VDD), LED123.1 (VDD), LED124.1 (VDD), LED125.1 (VDD), LED126.1 (VDD), LED127.1 (VDD), LED128.1 (VDD), LED129.1 (VDD), LED130.1 (VDD), LED131.1 (VDD), LED132.1 (VDD), LED133.1 (VDD), LED134.1 (VDD), LED135.1 (VDD), LED136.1 (VDD), LED137.1 (VDD), LED138.1 (VDD), LED139.1 (VDD), LED140.1 (VDD), LED141.1 (VDD), LED142.1 (VDD), LED143.1 (VDD), LED144.1 (VDD), LED97.1 (VDD), LED98.1 (VDD), LED99.1 (VDD), ShifterC5.1, ShifterC6.2, U10.23 (5V), U11.5 (VCC), U9.5 (VCC)
- net GND: now also C100.1, C101.1, C102.1, C103.1, C104.1, C105.1, C106.1, C107.1, C108.1, C109.1, C110.1, C111.1, C112.1, C113.1, C114.1, C115.1, C116.1, C117.1, C118.1, C119.1, C120.1, C121.1, C122.1, C123.1, C124.1, C125.1, C126.1, C127.1, C128.1, C129.1, C130.1, C131.1, C132.1, C133.1, C134.1, C135.1, C136.1, C137.1, C138.1, C139.1, C140.1, C141.1, C142.1, C143.1, C144.1, C97.1, C98.1, C99.1, ESD_C3.1, J3.A1 (GND), J3.A12 (GND), J3.B1 (GND), J3.B12 (GND), J3.S1 (SHIELD), LED100.4 (VSS), LED101.4 (VSS), LED102.4 (VSS), LED103.4 (VSS), LED104.4 (VSS), LED105.4 (VSS), LED106.4 (VSS), LED107.4 (VSS), LED108.4 (VSS), LED109.4 (VSS), LED110.4 (VSS), LED111.4 (VSS), LED112.4 (VSS), LED113.4 (VSS), LED114.4 (VSS), LED115.4 (VSS), LED116.4 (VSS), LED117.4 (VSS), LED118.4 (VSS), LED119.4 (VSS), LED120.4 (VSS), LED121.4 (VSS), LED122.4 (VSS), LED123.4 (VSS), LED124.4 (VSS), LED125.4 (VSS), LED126.4 (VSS), LED127.4 (VSS), LED128.4 (VSS), LED129.4 (VSS), LED130.4 (VSS), LED131.4 (VSS), LED132.4 (VSS), LED133.4 (VSS), LED134.4 (VSS), LED135.4 (VSS), LED136.4 (VSS), LED137.4 (VSS), LED138.4 (VSS), LED139.4 (VSS), LED140.4 (VSS), LED141.4 (VSS), LED142.4 (VSS), LED143.4 (VSS), LED144.4 (VSS), LED97.4 (VSS), LED98.4 (VSS), LED99.4 (VSS), ShifterC5.2, ShifterC6.1, U10.22 (GND), U11.1 (~{OE}), U11.3 (GND), U12.2 (VN), U9.1 (~{OE}), U9.3 (GND)
- net LINK+: now also J3.A6 (D+), J3.B6 (D+), JP5.2 (C), U12.6 (IO4)
- net LINK-: now also J3.A7 (D-), J3.B7 (D-), JP6.2 (C), U12.1 (IO1)
- net L_COL1: now also SW105.1, SW113.1, SW121.1, SW129.1, SW137.1, SW97.1, U10.10 (9)
- net L_COL2: now also SW106.1, SW114.1, SW122.1, SW130.1, SW138.1, SW98.1, U10.9 (8)
- net L_COL3: now also SW107.1, SW115.1, SW123.1, SW131.1, SW139.1, SW99.1, U10.8 (7)
- net L_COL4: now also SW100.1, SW108.1, SW116.1, SW124.1, SW132.1, SW140.1, U10.7 (6)
- net L_COL5: now also SW101.1, SW109.1, SW117.1, SW125.1, SW133.1, SW141.1, U10.6 (5)
- net L_COL6: now also SW102.1, SW110.1, SW118.1, SW126.1, SW134.1, SW142.1, U10.5 (4)
- net L_COL7: now also SW103.1, SW111.1, SW119.1, SW127.1, SW135.1, SW143.1, U10.4 (3)
- net L_COL8: now also SW104.1, SW112.1, SW120.1, SW128.1, SW136.1, SW144.1, U10.3 (2)
- net L_LED1: now also LED97.3 (DIN), R5.1
- net L_LED2: now also LED121.3 (DIN), R6.1
- net L_LED_3v3_1: now also U10.20 (29), U9.2 (A)
- net L_LED_3v3_2: now also U10.19 (28), U11.2 (A)
- net L_ROW1: now also D100.1 (K), D101.1 (K), D102.1 (K), D103.1 (K), D104.1 (K), D97.1 (K), D98.1 (K), D99.1 (K), U10.11 (10)
- net L_ROW2: now also D105.1 (K), D106.1 (K), D107.1 (K), D108.1 (K), D109.1 (K), D110.1 (K), D111.1 (K), D112.1 (K), U10.12 (11)
- net L_ROW3: now also D113.1 (K), D114.1 (K), D115.1 (K), D116.1 (K), D117.1 (K), D118.1 (K), D119.1 (K), D120.1 (K), U10.13 (12)
- net L_ROW4: now also D121.1 (K), D122.1 (K), D123.1 (K), D124.1 (K), D125.1 (K), D126.1 (K), D127.1 (K), D128.1 (K), U10.14 (13)
- net L_ROW5: now also D129.1 (K), D130.1 (K), D131.1 (K), D132.1 (K), D133.1 (K), D134.1 (K), D135.1 (K), D136.1 (K), U10.15 (14)
- net L_ROW6: now also D137.1 (K), D138.1 (K), D139.1 (K), D140.1 (K), D141.1 (K), D142.1 (K), D143.1 (K), D144.1 (K), U10.16 (15)
- net USART_RX: now also JP5.1 (A), JP6.1 (A), U10.2 (1)
- net USART_TX: now also JP5.3 (B), JP6.3 (B), U10.1 (0)
- net VSS_IN_FUSED: now also ESD_C3.2, J3.A4 (VBUS), J3.A9 (VBUS), J3.B4 (VBUS), J3.B9 (VBUS), U12.5 (VP)
- new net: D115.2 (A), SW115.2
- new net: D101.2 (A), SW101.2
- new net: D140.2 (A), SW140.2
- new net: LED100.2 (DOUT), LED101.3 (DIN)
- new net: LED100.3 (DIN), LED99.2 (DOUT)
- new net: LED138.2 (DOUT), LED139.3 (DIN)
- new net: LED137.2 (DOUT), LED138.3 (DIN)
- new net: D109.2 (A), SW109.2
- new net: D98.2 (A), SW98.2
- new net: D114.2 (A), SW114.2
- new net: D127.2 (A), SW127.2
- new net: R5.2, U9.4 (Y)
- new net: D119.2 (A), SW119.2
- new net: D126.2 (A), SW126.2
- new net: D135.2 (A), SW135.2
- new net: D106.2 (A), SW106.2
- new net: LED105.2 (DOUT), LED113.3 (DIN)
- new net: LED105.3 (DIN), LED106.2 (DOUT)
- new net: LED102.2 (DOUT), LED103.3 (DIN)
- new net: LED101.2 (DOUT), LED102.3 (DIN)
- new net: D102.2 (A), SW102.2
- new net: LED141.2 (DOUT), LED142.3 (DIN)
- new net: LED140.2 (DOUT), LED141.3 (DIN)
- new net: D124.2 (A), SW124.2
- new net: D122.2 (A), SW122.2
- new net: D117.2 (A), SW117.2
- new net: D110.2 (A), SW110.2
- new net: D97.2 (A), SW97.2
- new net: LED116.2 (DOUT), LED117.3 (DIN)
- new net: LED115.2 (DOUT), LED116.3 (DIN)
- new net: LED119.2 (DOUT), LED120.3 (DIN)
- new net: LED118.2 (DOUT), LED119.3 (DIN)
- new net: D121.2 (A), SW121.2
- new net: D105.2 (A), SW105.2
- new net: D144.2 (A), SW144.2
- new net: D107.2 (A), SW107.2
- new net: LED123.2 (DOUT), LED124.3 (DIN)
- new net: LED122.2 (DOUT), LED123.3 (DIN)
- new net: D139.2 (A), SW139.2
- new net: LED125.2 (DOUT), LED126.3 (DIN)
- new net: LED124.2 (DOUT), LED125.3 (DIN)
- new net: D108.2 (A), SW108.2
- new net: D118.2 (A), SW118.2
- new net: D136.2 (A), SW136.2
- new net: D132.2 (A), SW132.2
- new net: LED110.3 (DIN), LED111.2 (DOUT)
- new net: LED111.3 (DIN), LED112.2 (DOUT)
- new net: D137.2 (A), SW137.2
- new net: LED139.2 (DOUT), LED140.3 (DIN)
- new net: D130.2 (A), SW130.2
- new net: D120.2 (A), SW120.2
- new net: LED128.2 (DOUT), LED136.3 (DIN)
- new net: LED127.2 (DOUT), LED128.3 (DIN)
- new net: D125.2 (A), SW125.2
- new net: LED143.2 (DOUT), LED144.3 (DIN)
- new net: D99.2 (A), SW99.2
- new net: LED142.2 (DOUT), LED143.3 (DIN)
- new net: D141.2 (A), SW141.2
- new net: D134.2 (A), SW134.2
- new net: D138.2 (A), SW138.2
- new net: D133.2 (A), SW133.2
- new net: D112.2 (A), SW112.2
- new net: LED126.2 (DOUT), LED127.3 (DIN)
- new net: LED103.2 (DOUT), LED104.3 (DIN)
- new net: LED133.3 (DIN), LED134.2 (DOUT)
- new net: LED134.3 (DIN), LED135.2 (DOUT)
- new net: D142.2 (A), SW142.2
- new net: LED131.3 (DIN), LED132.2 (DOUT)
- new net: LED132.3 (DIN), LED133.2 (DOUT)
- new net: D128.2 (A), SW128.2
- new net: LED98.2 (DOUT), LED99.3 (DIN)
- new net: LED97.2 (DOUT), LED98.3 (DIN)
- new net: D113.2 (A), SW113.2
- new net: LED106.3 (DIN), LED107.2 (DOUT)
- new net: LED108.3 (DIN), LED109.2 (DOUT)
- new net: LED109.3 (DIN), LED110.2 (DOUT)
- new net: LED104.2 (DOUT), LED112.3 (DIN)
- new net: LED117.2 (DOUT), LED118.3 (DIN)
- new net: D116.2 (A), SW116.2
- new net: LED113.2 (DOUT), LED114.3 (DIN)
- new net: LED107.3 (DIN), LED108.2 (DOUT)
- new net: LED130.3 (DIN), LED131.2 (DOUT)
- new net: LED129.2 (DOUT), LED137.3 (DIN)
- new net: D143.2 (A), SW143.2
- new net: D100.2 (A), SW100.2
- new net: D123.2 (A), SW123.2
- new net: D103.2 (A), SW103.2
- new net: LED114.2 (DOUT), LED115.3 (DIN)
- new net: LED121.2 (DOUT), LED122.3 (DIN)
- new net: LED129.3 (DIN), LED130.2 (DOUT)
- new net: R6.2, U11.4 (Y)
- new net: D131.2 (A), SW131.2
- new net: D111.2 (A), SW111.2
- new net: LED135.3 (DIN), LED136.2 (DOUT)
- new net: D104.2 (A), SW104.2
- new net: D129.2 (A), SW129.2
- no-connect marks 11 -> 22
Other:
- moved on the sheet: C1, C10, C11, C12, C13, C14, C15, C16, C17, C18, C19, C2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
